File: HatsuLight69_left/HatsuLight69_left.kicad_pcb.kicad_pcb (KiCad board)
At the start: 2 copper layers, 12.8 x 6.7 mm, 139 parts, among them J1 USB_C_Receptacle, J2 MJ-4PP-9, J3 I2C, J4 SPI, SW1 SW_PUSH, SW10 SW_PUSH-kbd, SW11 SW_PUSH-kbd, SW12 SW_PUSH-kbd, SW13 SW_PUSH-kbd, SW14 SW_PUSH-kbd, SW15 SW_PUSH-kbd, SW16 SW_PUSH-kbd, SW17 SW_PUSH-kbd, SW18 SW_PUSH-kbd, SW19 SW_PUSH-kbd, SW2 SW_PUSH-kbd, SW20 SW_PUSH-kbd, SW21 SW_PUSH-kbd, SW22 SW_PUSH-kbd, SW23 SW_PUSH-kbd, SW24 SW_PUSH-kbd, SW25 SW_PUSH-kbd, SW26 SW_PUSH-kbd, SW27 SW_PUSH-kbd, SW28 SW_PUSH-kbd, SW29 SW_PUSH-kbd, SW3 SW_PUSH-kbd, SW30 SW_PUSH-kbd, SW31 SW_PUSH-kbd, SW32 SW_PUSH-kbd, SW33 SW_PUSH-kbd, SW34 SW_PUSH-kbd, SW35 SW_PUSH-kbd, SW36 SW_PUSH-kbd, SW37 SW_PUSH-kbd, SW38 SW_PUSH-kbd, SW4 SW_PUSH-kbd, SW5 SW_PUSH-kbd, SW6 SW_PUSH-kbd, SW7 SW_PUSH-kbd, SW8 SW_PUSH-kbd, SW9 SW_PUSH-kbd, U1 ATMEGA32U4, X1 CSTNE16M0V530000R0

Commit message: update
Parts:
- removed D68, D69, D70, D71, D72, D73, D74, D75, D76, D77: SK6812MINI, kbd:YS-SK6812MINI-E
- removed SW34, SW35, SW36, SW37, SW38: SW_PUSH-kbd, kbd:ChocV1_V2_Hotswap
- added ?: , , F.Cu at (50.0, 35.7)
- added ?: , , F.Cu at (196.5, 53.0)
- added ?: , , F.Cu at (126.2, 33.3)
- added ?: , , F.Cu at (50.0, 53.0)
- added ?: , , F.Cu at (126.2, 87.5)
- added REF**: MountingHole_2.2mm_M2, MountingHole:MountingHole_2.2mm_M2, F.Cu at (97.6, 53.0)
- added REF**: MountingHole_2.2mm_M2, MountingHole:MountingHole_2.2mm_M2, F.Cu at (69.1, 108.9)
- added REF**: MountingHole_2.2mm_M2, MountingHole:MountingHole_2.2mm_M2, F.Cu at (173.8, 53.0)
- added REF**: MountingHole_2.2mm_M2, MountingHole:MountingHole_2.2mm_M2, F.Cu at (184.5, 119.1)
- C1, C2, C3, C4, C5, C6, C7, D41, D42, D43, D44, D45, D46, D47, D48, D49, D50, D51, D52, D53, D54, D55, D56, D57, D58, D59, D60, D61, D62, D63, D64, D65, D66, D67, J4, R1, R10, R11, R2, R3, R4, R6, R7, U1, X1: moved to B.Cu
- D10, D11, D12, D13, D14, D15, D16, D17, D18, D19, D20, D21, D22, D23, D24, D25, D26, D27, D28, D29, D30, D31, D32, D33, D34, D35, D4, D5, D6, D7, D8, D9: footprint kbd:D3_SMD -> kbd:D3_SMD_v2; moved to B.Cu
- D36, D37, D38, D39, D40: value D_Small -> SK6812MINI; footprint kbd:D3_SMD -> kbd:YS-SK6812MINI-E; moved to B.Cu
- R5, R8, R9: value 1k -> 1000
- SW16, SW33: footprint kbd:ChocV1_V2_Hotswap -> kbd:ChocV1_V2_Hotswap_2u
- SW22: footprint kbd:ChocV1_V2_Hotswap -> kbd:ChocV1_V2_Hotswap_2.5u
- SW31, SW9: footprint kbd:ChocV1_V2_Hotswap -> kbd:ChocV1_V2_Hotswap_1.5u
- moved D36 376.3 mm to (194.5, 136.0), turned to -135 degrees
- moved SW27 348.3 mm to (183.4, 98.8), turned to 180 degrees
- moved D35 347.4 mm to (185.1, 138.7), turned to 135 degrees
- moved SW26 345.8 mm to (164.3, 98.8), turned to 180 degrees
- moved SW15 345.7 mm to (183.4, 60.7), turned to 180 degrees
- moved SW8 336.1 mm to (173.8, 41.7)
- moved D29 331.3 mm to (175.0, 100.0), turned to 90 degrees
- moved D22 330.8 mm to (146.4, 81.0), turned to 90 degrees
- moved D9 330.4 mm to (163.1, 40.5), turned to 90 degrees
- moved D8 329.6 mm to (144.1, 40.5), turned to 90 degrees
- moved D17 329.6 mm to (175.0, 61.9), turned to 90 degrees
- moved D37 326.9 mm to (158.1, 130.3), turned to 165 degrees
- moved D27 325.9 mm to (136.9, 100.0), turned to 90 degrees
- moved D10 324.3 mm to (165.5, 40.5), turned to 90 degrees
- moved D23 324.0 mm to (165.5, 81.0), turned to 90 degrees
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Connections:
- D18 pad 1: ROW1 -> ROW2
- D24 pad 1: ROW2 -> ROW3
- D25 pad 1: ROW2 -> ROW3
- D30 pad 1: ROW3 -> ROW4
- D31 pad 1: ROW3 -> ROW4
- D32 pad 1: ROW3 -> ROW4
- D33 pad 1: ROW3 -> ROW4
- D36 pad 1: ROW4 -> Net-(D36-Pad1)
- D36 pad 2: Net-(D36-Pad2) -> GND
- D37 pad 1: ROW4 -> Net-(D37-Pad1)
- D37 pad 2: Net-(D37-Pad2) -> GND
- D38 pad 1: ROW4 -> Net-(D38-Pad1)
- D38 pad 2: Net-(D38-Pad2) -> GND
- D39 pad 1: ROW4 -> Net-(D39-Pad1)
- D39 pad 2: Net-(D39-Pad2) -> GND
- D40 pad 1: ROW4 -> Net-(D40-Pad1)
- D40 pad 2: Net-(D40-Pad2) -> GND
- D41 pad 3: LED -> Net-(D40-Pad1)
- D67 pad 1: Net-(D67-Pad1) -> unconnected-(D67-Pad1)
- J1 pad A3: unconnected-(J1-PadA3) -> (no net)
- J1 pad A6: Net-(J1-PadA6) -> (no net)
- J1 pad A7: Net-(J1-PadA7) -> (no net)
- SW16 pad 1: COL7 -> COL0
- SW17 pad 1: COL0 -> COL1
- SW18 pad 1: COL1 -> COL2
- SW19 pad 1: COL2 -> COL3
- SW20 pad 1: COL3 -> COL4
- SW21 pad 1: COL4 -> COL5
- SW22 pad 1: COL5 -> COL0
- SW23 pad 1: COL6 -> COL1
- SW24 pad 1: COL0 -> COL2
- SW25 pad 1: COL1 -> COL3
- SW26 pad 1: COL2 -> COL4
- SW27 pad 1: COL3 -> COL5
- SW28 pad 1: COL4 -> COL0
- SW29 pad 1: COL5 -> COL1
- SW30 pad 1: COL6 -> COL2
- SW31 pad 1: COL7 -> COL3
- SW32 pad 1: COL0 -> COL4
- SW33 pad 1: COL1 -> COL5
- SW8 pad 1: COL6 -> Net-(D10-Pad2)
- SW8 pad 2: Net-(D10-Pad2) -> COL6
- U1 pad 25: COL7 -> unconnected-(U1-Pad25)
Routing:
- net VCC: track 0.00 -> 1088.7 mm, vias 0 -> 25
- net COL0: track 0.00 -> 215.6 mm, vias 0 -> 10
- net COL1: track 0.00 -> 206.6 mm, vias 0 -> 10
- net ROW4: track 0.00 -> 203.8 mm, vias 0 -> 2
- net COL2: track 0.00 -> 184.1 mm, vias 0 -> 10
- net ROW0: track 0.00 -> 182.3 mm, vias 0 -> 2
- net COL3: track 0.00 -> 161.0 mm, vias 0 -> 10
- net MISO: track 0.00 -> 157.1 mm, vias 0 -> 4
- net MOSI: track 0.00 -> 154.9 mm, vias 0 -> 4
- net ROW3: track 0.00 -> 144.9 mm, vias 0 -> 2
- net SCLK: track 0.00 -> 141.2 mm, vias 0 -> 4
- net NCS: track 0.00 -> 140.0 mm, vias 0 -> 4
- net ROW1: track 0.00 -> 138.2 mm, vias 0 -> 2
- net ROW2: track 0.00 -> 138.2 mm, vias 0 -> 2
- net COL4: track 0.00 -> 133.6 mm, vias 0 -> 8
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- added copper zone on B.Cu, net GND
- added copper zone on F.Cu, net GND
Other:
- board size 12.8 x 6.7 mm -> 164.5 x 124 mm
- board text added: "0.1u"
- board text added: "1"
- board text added: "10"
- board text added: "10k"
- board text added: "11"
- board text added: "12"
- board text added: "13"
- board text added: "14"
- board text added: "15"
- board text added: "16"
- board text added: "17"
- board text added: "18"
- board text added: "19"
- board text added: "1u"
- board text added: "2"
- board text added: "20"
- board text added: "21"
- board text added: "22"
- board text added: "23"
- board text added: "24"
- board text added: "25"
- board text added: "26"
- board text added: "27"
- board text added: "28"
- board text added: "29"
- board text added: "3"
- board text added: "30"
- board text added: "31"
- board text added: "32"
- board text added: "4"
- board text added: "4.7u"
- board text added: "5"
- board text added: "5.1k"
- board text added: "5V"
- board text added: "6"
- board text added: "7"
- board text added: "8"
- board text added: "9"
- board text added: "CLK"
- board text added: "CS"
- board text added: "G"
- board text added: "HatsuLight rev0.1"
- board text added: "MI SO"
- board text added: "MO SI"
- board text added: "OLED"
- board text added: "SPI"
- board text added: "designed by"
- board text added: "driving="
- board text added: "hearing="
- board text added: "kazmeegawa"
- board text added: "talking="

Commit message: update
Other:
- board size 164.5 x 124 mm -> 164.5 x 123.6 mm
Changed lines of the file:
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@@
   (gr_line (start 47.62514 35.71886) (end 47.62514 125.01581) (layer "Edge.Cuts") (width 0.1))
   (gr_arc (start 212.119649 124.389144) (mid 212.048446 125.976583) (end 211.336215 127.397062) (layer "Edge.Cuts") (width 0.1))
-  (gr_line (start 170.27102 141.076908) (end 182.165878 152.995521) (layer "Edge.Cuts") (width 0.1))
   (gr_arc (start 133.945525 130.96894) (mid 136.350312 131.090679) (end 138.730511 131.454651) (layer "Edge.Cuts") (width 0.1))
-  (gr_line (start 185.737756 152.995521) (end 211.336215 127.397062) (layer "Edge.Cuts") (width 0.1))
   (gr_arc (start 191.690886 29.76573) (mid 194.842723 30.957889) (end 196.416613 33.937518) (layer "Edge.Cuts") (width 0.1))
+  (gr_line (start 170.27102 141.076908) (end 181.349466 152.177417) (layer "Edge.Cuts") (width 0.1))
   (gr_line (start 191.542443 29.765732) (end 191.003069 29.765732) (layer "Edge.Cuts") (width 0.1))
   (gr_arc (start 166.092427 138.708009) (mid 168.318349 139.651459) (end 170.27102 141.076908) (layer "Edge.Cuts") (width 0.1))
+  (gr_arc (start 186.512199 152.222199) (mid 183.92113 153.318406) (end 181.349466 152.177417) (layer "Edge.Cuts") (width 0.1))
   (gr_arc (start 53.57827 130.96894) (mid 49.368771 129.225309) (end 47.62514 125.01581) (layer "Edge.Cuts") (width 0.1))
-  (gr_arc (start 185.737756 152.995521) (mid 183.951817 153.735281) (end 182.165878 152.995521) (layer "Edge.Cuts") (width 0.1))
   (gr_line (start 179.933069 29.765732) (end 53.57827 29.76573) (layer "Edge.Cuts") (width 0.1))
   (gr_line (start 130.96896 130.96894) (end 133.945525 130.96894) (layer "Edge.Cuts") (width 0.1))
   (gr_line (start 191.542443 29.765732) (end 191.690886 29.76573) (layer "Edge.Cuts") (width 0.1))
+  (gr_line (start 186.512199 152.222199) (end 211.336215 127.397062) (layer "Edge.Cuts") (width 0.1))
   (gr_line (start 53.57827 130.96894) (end 130.96896 130.96894) (layer "Edge.Cuts") (width 0.1))
   (gr_arc (start 47.62514 35.71886) (mid 49.368771 31.509361) (end 53.57827 29.76573) (layer "Edge.Cuts") (width 0.1))

Commit message: update
Parts:
- D1, D2, D3, R5, R8, R9: moved to B.Cu
- J3: footprint Connector_PinHeader_2.54mm:PinHeader_1x04_P2.54mm_Vertical -> kbd:OLED_v2
- moved J4 55.8 mm to (145.8, 128.6), turned to -15 degrees
- moved ? 3.57 mm to (50.0, 32.1)
- moved J3 3.50 mm to (203.3, 106.8), turned to 10 degrees
- moved R4 3.33 mm to (190.3, 40.2), turned to 0 degrees
- moved D1 2.68 mm to (206.5, 95.0)
- moved D2 2.64 mm to (206.9, 96.7)
- moved D3 2.62 mm to (207.4, 98.3)
- moved R1 2.57 mm to (186.9, 41.4), turned to 180 degrees
- moved R3 2.33 mm to (190.3, 41.4), turned to 0 degrees
- moved J1 2.26 mm to (188.6, 32.1)
- moved R8 1.92 mm to (202.2, 97.2)
- moved R9 1.92 mm to (202.2, 98.9)
- moved R5 1.92 mm to (202.2, 95.4)
- moved ? 1.79 mm to (50.0, 51.2)
- moved J2 1.39 mm to (197.6, 44.7)
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Connections:
- J1 pad A6: (no net) -> Net-(J1-PadA6)
- J1 pad A7: (no net) -> Net-(J1-PadA7)
- J3 pad 1: VCC -> SDA
- J3 pad 2: GND -> SCL
- J3 pad 3: SCL -> VCC
- J3 pad 4: SDA -> GND
Routing:
- net SCLK: track 141.2 -> 79.6 mm, vias 4 -> 2
- net MISO: track 157.1 -> 96.0 mm, vias 4 -> 2
- net MOSI: track 154.9 -> 94.4 mm, vias 4 -> 2
- net NCS: track 140.0 -> 79.7 mm, vias 4 -> 2
- net VCC: track 1088.7 -> 1052.4 mm, vias 25 -> 23
- net /MCU/D+: track 44.9 -> 50.6 mm
- net SDA: track 27.8 -> 22.4 mm
- net Net-(J1-PadA7): track 3.59 -> 8.58 mm, vias 0 -> 2
- net SCL: track 28.1 -> 23.6 mm
- net ROW4: track 203.8 -> 208.0 mm
- net Net-(R8-Pad2): track 17.0 -> 13.7 mm, vias 1 -> 2
- net Net-(J1-PadA6): track 3.42 -> 6.66 mm, vias 0 -> 2
- net /MCU/D-: track 45.6 -> 48.2 mm
- net ROW0: track 182.3 -> 180.6 mm
- net Net-(D37-Pad1): track 33.5 -> 35.0 mm
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Other:
- board size 164.5 x 123.6 mm -> 166.3 x 125.7 mm
- board text added: "=driving"
- board text added: "=hearing"
- board text added: "=talking"
- board text removed: "OLED"
- board text removed: "driving="
- board text removed: "hearing="
- board text removed: "talking="
