File: HatsuLight69_left/HatsuLight69_left.kicad_pcb.kicad_pcb (KiCad board)
At the start: 2 copper layers, 166.3 x 125.7 mm, 133 parts, among them J1 USB_C_Receptacle, J2 MJ-4PP-9, J3 I2C, J4 SPI, SW1 SW_PUSH, SW10 SW_PUSH-kbd, SW11 SW_PUSH-kbd, SW12 SW_PUSH-kbd, SW13 SW_PUSH-kbd, SW14 SW_PUSH-kbd, SW15 SW_PUSH-kbd, SW16 SW_PUSH-kbd, SW17 SW_PUSH-kbd, SW18 SW_PUSH-kbd, SW19 SW_PUSH-kbd, SW2 SW_PUSH-kbd, SW20 SW_PUSH-kbd, SW21 SW_PUSH-kbd, SW22 SW_PUSH-kbd, SW23 SW_PUSH-kbd, SW24 SW_PUSH-kbd, SW25 SW_PUSH-kbd, SW26 SW_PUSH-kbd, SW27 SW_PUSH-kbd, SW28 SW_PUSH-kbd, SW29 SW_PUSH-kbd, SW3 SW_PUSH-kbd, SW30 SW_PUSH-kbd, SW31 SW_PUSH-kbd, SW32 SW_PUSH-kbd, SW33 SW_PUSH-kbd, SW4 SW_PUSH-kbd, SW5 SW_PUSH-kbd, SW6 SW_PUSH-kbd, SW7 SW_PUSH-kbd, SW8 SW_PUSH-kbd, SW9 SW_PUSH-kbd, U1 ATMEGA32U4, X1 CSTNE16M0V530000R0

Commit message: update
Parts:
- J1: moved to B.Cu
- turned J1 to 0 degrees
Routing:
- net Net-(J1-PadB5): track 3.30 -> 5.81 mm, vias 0 -> 1
- net Net-(J1-PadA5): track 5.33 -> 4.26 mm, vias 1 -> 0
- net unconnected-(J1-PadA8): track 0.00 -> 0.50 mm
- net Net-(J1-PadA6): track 6.66 -> 6.69 mm, vias 2 -> 1
Other:
- outline, holes or cut-outs redrawn

Commit message: update
Parts:
- R5, R8, R9: value 1000 -> 1k
Connections:
- J1 pad A3: (no net) -> unconnected-(J1-PadA3)
- J3 pad 1: SDA -> VCC
- J3 pad 2: SCL -> GND
- J3 pad 3: VCC -> SCL
- J3 pad 4: GND -> SDA
- SW8 pad 1: Net-(D10-Pad2) -> COL6
- SW8 pad 2: COL6 -> Net-(D10-Pad2)
Changed lines of the file:
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@@
       (drillshape 0)
       (scaleselection 1)
-      (outputdirectory "gbr/")
+      (outputdirectory "pos/")
     )
   )
@@
   (net 74 "Net-(D40-Pad1)")
   (net 75 "unconnected-(U1-Pad25)")
-  (net 76 "Net-(D50-Pad3)")
-  (net 77 "Net-(D62-Pad3)")
+  (net 76 "Net-(D49-Pad1)")
+  (net 77 "Net-(D61-Pad1)")
   (net 78 "unconnected-(J1-PadA2)")
   (net 79 "Net-(J1-PadA5)")
@@
   (net 114 "DATA")
   (net 115 "unconnected-(D67-Pad1)")
+  (net 116 "unconnected-(J1-PadA3)")
   (footprint "kbd:ChocV1_V2_Hotswap" (layer "F.Cu")
     (at 135.7313 41.67191)
@@
     (pad "" np_thru_hole circle (at 0 0 90) (size 5 5) (drill 5) (layers *.Cu))
     (pad "1" smd rect (at -8.3 3.7 180) (size 2.6 2.6) (layers "B.Cu" "B.Paste" "B.Mask")
-      (net 15 "Net-(D10-Pad2)") (pinfunction "1") (pintype "passive"))
+      (net 109 "COL6") (pinfunction "1") (pintype "passive"))
     (pad "2" smd rect (at 3.3 5.9 180) (size 2.6 2.6) (layers "B.Cu" "B.Paste" "B.Mask")
-      (net 109 "COL6") (pinfunction "2") (pintype "passive"))
+      (net 15 "Net-(D10-Pad2)") (pinfunction "2") (pintype "passive"))
     (model "${KIPRJMOD}/parts/kbd/kicad-packages3D/kbd.3dshapes/kailh_choc.step"
       (offset (xyz 0 0 0))
@@
     (fp_line (start -6 -36.73) (end 6 -36.73) (layer "Dwgs.User") (width 0.12))
     (pad "1" thru_hole circle (at -3.810001 0 10) (size 1.397 1.397) (drill 0.8128) (layers *.Cu "F.SilkS" "B.Mask")
-      (net 92 "SDA") (pinfunction "Pin_1") (pintype "passive"))
+      (net 4 "VCC") (pinfunction "Pin_1") (pintype "passive"))
     (pad "2" thru_hole circle (at -1.27 0 10) (size 1.397 1.397) (drill 0.8128) (layers *.Cu "F.SilkS" "B.Mask")
-      (net 91 "SCL") (pinfunction "Pin_2") (pintype "passive"))
+      (net 2 "GND") (pinfunction "Pin_2") (pintype "passive"))
     (pad "3" thru_hole circle (at 1.27 0 10) (size 1.397 1.397) (drill 0.8128) (layers *.Cu "F.SilkS" "B.Mask")
-      (net 4 "VCC") (pinfunction "Pin_3") (pintype "passive"))
+      (net 91 "SCL") (pinfunction "Pin_3") (pintype "passive"))
     (pad "4" thru_hole circle (at 3.810001 0 10) (size 1.397 1.397) (drill 0.8128) (layers *.Cu "F.SilkS" "B.Mask")
-      (net 2 "GND") (pinfunction "Pin_4") (pintype "passive"))
+      (net 92 "SDA") (pinfunction "Pin_4") (pintype "passive"))
     (model "${KIPRJMOD}/parts/kbd/kicad-packages3D/kbd.3dshapes/OLED-Module-with-Pins.step"
       (offset (xyz 0 0 0))
@@
       (net 78 "unconnected-(J1-PadA2)") (pinfunction "TX1+") (pintype "bidirectional+no_connect"))
     (pad "A3" smd rect (at -1.4 5.74375 270) (size 0.85 0.23) (layers "B.Cu" "B.Paste" "B.Mask")
-      (pinfunction "TX1-") (pintype "bidirectional+no_connect"))
+      (net 116 "unconnected-(J1-PadA3)") (pinfunction "TX1-") (pintype "bidirectional+no_connect"))
     (pad "A4" smd rect (at -1 5.74375 270) (size 0.85 0.23) (layers "B.Cu" "B.Paste" "B.Mask")
       (net 4 "VCC") (pinfunction "VBUS") (pintype "passive"))
@@
       (effects (font (size 1 1) (thickness 0.15)) (justify mirror))
     )
-    (fp_text value "1000" (at 3.33375 0) (layer "B.SilkS")
+    (fp_text value "1k" (at 3.33375 0) (layer "B.SilkS")
       (effects (font (size 1 1) (thickness 0.15)) (justify mirror))
     )
@@
       (net 2 "GND") (pinfunction "VSS") (pintype "power_in"))
     (pad "3" smd rect (at -2.75 -0.7 180) (size 1.7 1) (layers "B.Cu" "B.Paste" "B.Mask")
-      (net 77 "Net-(D62-Pad3)") (pinfunction "DIN") (pintype "input"))
+      (net 77 "Net-(D61-Pad1)") (pinfunction "DIN") (pintype "input"))
     (pad "4" smd rect (at -2.75 0.7 180) (size 1.7 1) (layers "B.Cu" "B.Paste" "B.Mask")
       (net 4 "VCC") (pinfunction "VDD") (pintype "power_in"))
@@
       (net 2 "GND") (pinfunction "VSS") (pintype "power_in"))
     (pad "3" smd rect (at -2.75 -0.7 180) (size 1.7 1) (layers "B.Cu" "B.Paste" "B.Mask")
-      (net 76 "Net-(D50-Pad3)") (pinfunction "DIN") (pintype "input"))
+      (net 76 "Net-(D49-Pad1)") (pinfunction "DIN") (pintype "input"))
     (pad "4" smd rect (at -2.75 0.7 180) (size 1.7 1) (layers "B.Cu" "B.Paste" "B.Mask")
       (net 4 "VCC") (pinfunction "VDD") (pintype "power_in"))
@@
       (effects (font (size 1 1) (thickness 0.15)) (justify mirror))
     )
-    (fp_text value "1000" (at 3.33375 -0.119064) (layer "B.SilkS")
+    (fp_text value "1k" (at 3.33375 -0.119064) (layer "B.SilkS")
       (effects (font (size 1 1) (thickness 0.15)) (justify mirror))
     )
@@
     (fp_line (start -1.8 1.55) (end -1.8 -1.55) (layer "Edge.Cuts") (width 0.12))
     (pad "1" smd rect (at 2.75 0.7 180) (size 1.7 1) (layers "B.Cu" "B.Paste" "B.Mask")
-      (net 77 "Net-(D62-Pad3)") (pinfunction "DOUT") (pintype "output"))
+      (net 77 "Net-(D61-Pad1)") (pinfunction "DOUT") (pintype "output"))
     (pad "2" smd rect (at 2.75 -0.7 180) (size 1.7 1) (layers "B.Cu" "B.Paste" "B.Mask")
       (net 2 "GND") (pinfunction "VSS") (pintype "power_in"))
@@
       (effects (font (size 1 1) (thickness 0.15)) (justify mirror))
     )
-    (fp_text value "1000" (at -3.33375 0) (layer "B.SilkS")
+    (fp_text value "1k" (at -3.33375 0) (layer "B.SilkS")
       (effects (font (size 1 1) (thickness 0.15)) (justify mirror))
     )
@@
     (fp_line (start -1.8 1.55) (end -1.8 -1.55) (layer "Edge.Cuts") (width 0.12))
     (pad "1" smd rect (at 2.75 0.7 180) (size 1.7 1) (layers "B.Cu" "B.Paste" "B.Mask")
-      (net 76 "Net-(D50-Pad3)") (pinfunction "DOUT") (pintype "output"))
+      (net 76 "Net-(D49-Pad1)") (pinfunction "DOUT") (pintype "output"))
     (pad "2" smd rect (at 2.75 -0.7 180) (size 1.7 1) (layers "B.Cu" "B.Paste" "B.Mask")
       (net 2 "GND") (pinfunction "VSS") (pintype "power_in"))
