File: HatsuLight69_left/key_switch.kicad_sch (KiCad schematic)
At the start: 64 parts, among them SW10 SW_PUSH-kbd, SW11 SW_PUSH-kbd, SW12 SW_PUSH-kbd, SW13 SW_PUSH-kbd, SW14 SW_PUSH-kbd, SW15 SW_PUSH-kbd, SW16 SW_PUSH-kbd, SW17 SW_PUSH-kbd, SW18 SW_PUSH-kbd, SW19 SW_PUSH-kbd, SW2 SW_PUSH-kbd, SW20 SW_PUSH-kbd, SW21 SW_PUSH-kbd, SW22 SW_PUSH-kbd, SW23 SW_PUSH-kbd, SW24 SW_PUSH-kbd, SW25 SW_PUSH-kbd, SW26 SW_PUSH-kbd, SW27 SW_PUSH-kbd, SW28 SW_PUSH-kbd, SW29 SW_PUSH-kbd, SW3 SW_PUSH-kbd, SW30 SW_PUSH-kbd, SW31 SW_PUSH-kbd, SW32 SW_PUSH-kbd, SW33 SW_PUSH-kbd, SW4 SW_PUSH-kbd, SW5 SW_PUSH-kbd, SW6 SW_PUSH-kbd, SW7 SW_PUSH-kbd, SW8 SW_PUSH-kbd, SW9 SW_PUSH-kbd

Commit message: update
Parts:
- D10, D11, D12, D13, D14, D15, D16, D17, D18, D19, D20, D21, D22, D23, D24, D25, D26, D27, D28, D29, D30, D31, D32, D33, D34, D35, D4, D5, D6, D7, D8, D9: footprint kbd:D3_SMD_v2 -> kbd:D3_SMD
Changed lines of the file:
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@@
       (effects (font (size 1.27 1.27)) (justify right) hide)
     )
-    (property "Footprint" "kbd:D3_SMD_v2" (id 2) (at 146.05 95.25 90)
+    (property "Footprint" "kbd:D3_SMD" (id 2) (at 146.05 95.25 90)
       (effects (font (size 1.27 1.27)) hide)
     )
@@
       (effects (font (size 1.27 1.27)) (justify right) hide)
     )
-    (property "Footprint" "kbd:D3_SMD_v2" (id 2) (at 146.05 135.89 90)
+    (property "Footprint" "kbd:D3_SMD" (id 2) (at 146.05 135.89 90)
       (effects (font (size 1.27 1.27)) hide)
     )
@@
       (effects (font (size 1.27 1.27)) (justify right) hide)
     )
-    (property "Footprint" "kbd:D3_SMD_v2" (id 2) (at 123.19 135.89 90)
+    (property "Footprint" "kbd:D3_SMD" (id 2) (at 123.19 135.89 90)
       (effects (font (size 1.27 1.27)) hide)
     )
@@
       (effects (font (size 1.27 1.27)) (justify right) hide)
     )
-    (property "Footprint" "kbd:D3_SMD_v2" (id 2) (at 100.33 95.25 90)
+    (property "Footprint" "kbd:D3_SMD" (id 2) (at 100.33 95.25 90)
       (effects (font (size 1.27 1.27)) hide)
     )
@@
       (effects (font (size 1.27 1.27)) (justify right) hide)
     )
-    (property "Footprint" "kbd:D3_SMD_v2" (id 2) (at 168.91 135.89 90)
+    (property "Footprint" "kbd:D3_SMD" (id 2) (at 168.91 135.89 90)
       (effects (font (size 1.27 1.27)) hide)
     )
@@
       (effects (font (size 1.27 1.27)) (justify right) hide)
     )
-    (property "Footprint" "kbd:D3_SMD_v2" (id 2) (at 77.47 135.89 90)
+    (property "Footprint" "kbd:D3_SMD" (id 2) (at 77.47 135.89 90)
       (effects (font (size 1.27 1.27)) hide)
     )
@@
       (effects (font (size 1.27 1.27)) (justify right) hide)
     )
-    (property "Footprint" "kbd:D3_SMD_v2" (id 2) (at 146.05 54.61 90)
+    (property "Footprint" "kbd:D3_SMD" (id 2) (at 146.05 54.61 90)
       (effects (font (size 1.27 1.27)) hide)
     )
@@
       (effects (font (size 1.27 1.27)) (justify right) hide)
     )
-    (property "Footprint" "kbd:D3_SMD_v2" (id 2) (at 100.33 135.89 90)
+    (property "Footprint" "kbd:D3_SMD" (id 2) (at 100.33 135.89 90)
       (effects (font (size 1.27 1.27)) hide)
     )
@@
       (effects (font (size 1.27 1.27)) (justify right) hide)
     )
-    (property "Footprint" "kbd:D3_SMD_v2" (id 2) (at 123.19 95.25 90)
+    (property "Footprint" "kbd:D3_SMD" (id 2) (at 123.19 95.25 90)
       (effects (font (size 1.27 1.27)) hide)
     )
@@
       (effects (font (size 1.27 1.27)) (justify right) hide)
     )
-    (property "Footprint" "kbd:D3_SMD_v2" (id 2) (at 214.63 74.93 90)
+    (property "Footprint" "kbd:D3_SMD" (id 2) (at 214.63 74.93 90)
       (effects (font (size 1.27 1.27)) hide)
     )
@@
       (effects (font (size 1.27 1.27)) (justify right) hide)
     )
-    (property "Footprint" "kbd:D3_SMD_v2" (id 2) (at 168.91 115.57 90)
+    (property "Footprint" "kbd:D3_SMD" (id 2) (at 168.91 115.57 90)
       (effects (font (size 1.27 1.27)) hide)
     )
@@
       (effects (font (size 1.27 1.27)) (justify right) hide)
     )
-    (property "Footprint" "kbd:D3_SMD_v2" (id 2) (at 100.33 74.93 90)
+    (property "Footprint" "kbd:D3_SMD" (id 2) (at 100.33 74.93 90)
       (effects (font (size 1.27 1.27)) hide)
     )
@@
       (effects (font (size 1.27 1.27)) (justify right) hide)
     )
-    (property "Footprint" "kbd:D3_SMD_v2" (id 2) (at 77.47 74.93 90)
+    (property "Footprint" "kbd:D3_SMD" (id 2) (at 77.47 74.93 90)
       (effects (font (size 1.27 1.27)) hide)
     )
@@
       (effects (font (size 1.27 1.27)) (justify right) hide)
     )
-    (property "Footprint" "kbd:D3_SMD_v2" (id 2) (at 191.77 95.25 90)
+    (property "Footprint" "kbd:D3_SMD" (id 2) (at 191.77 95.25 90)
       (effects (font (size 1.27 1.27)) hide)
     )
@@
       (effects (font (size 1.27 1.27)) (justify right) hide)
     )
-    (property "Footprint" "kbd:D3_SMD_v2" (id 2) (at 123.19 74.93 90)
+    (property "Footprint" "kbd:D3_SMD" (id 2) (at 123.19 74.93 90)
       (effects (font (size 1.27 1.27)) hide)
     )
@@
       (effects (font (size 1.27 1.27)) (justify right) hide)
     )
-    (property "Footprint" "kbd:D3_SMD_v2" (id 2) (at 100.33 115.57 90)
+    (property "Footprint" "kbd:D3_SMD" (id 2) (at 100.33 115.57 90)
       (effects (font (size 1.27 1.27)) hide)
     )
@@
       (effects (font (size 1.27 1.27)) (justify right) hide)
     )
-    (property "Footprint" "kbd:D3_SMD_v2" (id 2) (at 146.05 74.93 90)
+    (property "Footprint" "kbd:D3_SMD" (id 2) (at 146.05 74.93 90)
       (effects (font (size 1.27 1.27)) hide)
     )
@@
       (effects (font (size 1.27 1.27)) (justify right) hide)
     )
-    (property "Footprint" "kbd:D3_SMD_v2" (id 2) (at 168.91 54.61 90)
+    (property "Footprint" "kbd:D3_SMD" (id 2) (at 168.91 54.61 90)
       (effects (font (size 1.27 1.27)) hide)
     )
@@
       (effects (font (size 1.27 1.27)) (justify right) hide)
     )
-    (property "Footprint" "kbd:D3_SMD_v2" (id 2) (at 77.47 95.25 90)
+    (property "Footprint" "kbd:D3_SMD" (id 2) (at 77.47 95.25 90)
       (effects (font (size 1.27 1.27)) hide)
     )
@@
       (effects (font (size 1.27 1.27)) (justify right) hide)
     )
-    (property "Footprint" "kbd:D3_SMD_v2" (id 2) (at 191.77 74.93 90)
+    (property "Footprint" "kbd:D3_SMD" (id 2) (at 191.77 74.93 90)
       (effects (font (size 1.27 1.27)) hide)
     )
@@
       (effects (font (size 1.27 1.27)) (justify right) hide)
     )
-    (property "Footprint" "kbd:D3_SMD_v2" (id 2) (at 123.19 54.61 90)
+    (property "Footprint" "kbd:D3_SMD" (id 2) (at 123.19 54.61 90)
       (effects (font (size 1.27 1.27)) hide)
     )
@@
       (effects (font (size 1.27 1.27)) (justify right) hide)
     )
-    (property "Footprint" "kbd:D3_SMD_v2" (id 2) (at 191.77 135.89 90)
+    (property "Footprint" "kbd:D3_SMD" (id 2) (at 191.77 135.89 90)
       (effects (font (size 1.27 1.27)) hide)
     )
@@
       (effects (font (size 1.27 1.27)) (justify right) hide)
     )
-    (property "Footprint" "kbd:D3_SMD_v2" (id 2) (at 214.63 54.61 90)
+    (property "Footprint" "kbd:D3_SMD" (id 2) (at 214.63 54.61 90)
       (effects (font (size 1.27 1.27)) hide)
     )
@@
       (effects (font (size 1.27 1.27)) (justify right) hide)
     )
-    (property "Footprint" "kbd:D3_SMD_v2" (id 2) (at 146.05 115.57 90)
+    (property "Footprint" "kbd:D3_SMD" (id 2) (at 146.05 115.57 90)
       (effects (font (size 1.27 1.27)) hide)
     )
@@
       (effects (font (size 1.27 1.27)) (justify right) hide)
     )
-    (property "Footprint" "kbd:D3_SMD_v2" (id 2) (at 168.91 95.25 90)
+    (property "Footprint" "kbd:D3_SMD" (id 2) (at 168.91 95.25 90)
       (effects (font (size 1.27 1.27)) hide)
     )
@@
       (effects (font (size 1.27 1.27)) (justify right) hide)
     )
-    (property "Footprint" "kbd:D3_SMD_v2" (id 2) (at 77.47 54.61 90)
+    (property "Footprint" "kbd:D3_SMD" (id 2) (at 77.47 54.61 90)
       (effects (font (size 1.27 1.27)) hide)
     )
@@
       (effects (font (size 1.27 1.27)) (justify right) hide)
     )
-    (property "Footprint" "kbd:D3_SMD_v2" (id 2) (at 123.19 115.57 90)
+    (property "Footprint" "kbd:D3_SMD" (id 2) (at 123.19 115.57 90)
       (effects (font (size 1.27 1.27)) hide)
     )
@@
       (effects (font (size 1.27 1.27)) (justify right) hide)
     )
-    (property "Footprint" "kbd:D3_SMD_v2" (id 2) (at 191.77 54.61 90)
+    (property "Footprint" "kbd:D3_SMD" (id 2) (at 191.77 54.61 90)
       (effects (font (size 1.27 1.27)) hide)
     )
@@
       (effects (font (size 1.27 1.27)) (justify right) hide)
     )
-    (property "Footprint" "kbd:D3_SMD_v2" (id 2) (at 168.91 74.93 90)
+    (property "Footprint" "kbd:D3_SMD" (id 2) (at 168.91 74.93 90)
       (effects (font (size 1.27 1.27)) hide)
     )
@@
       (effects (font (size 1.27 1.27)) (justify right) hide)
     )
-    (property "Footprint" "kbd:D3_SMD_v2" (id 2) (at 100.33 54.61 90)
+    (property "Footprint" "kbd:D3_SMD" (id 2) (at 100.33 54.61 90)
       (effects (font (size 1.27 1.27)) hide)
     )
@@
       (effects (font (size 1.27 1.27)) (justify right) hide)
     )
-    (property "Footprint" "kbd:D3_SMD_v2" (id 2) (at 77.47 115.57 90)
+    (property "Footprint" "kbd:D3_SMD" (id 2) (at 77.47 115.57 90)
       (effects (font (size 1.27 1.27)) hide)
     )
@@
       (effects (font (size 1.27 1.27)) (justify right) hide)
     )
-    (property "Footprint" "kbd:D3_SMD_v2" (id 2) (at 191.77 115.57 90)
-      (effects (font (size 1.27 1.27)) hide)
-    )
+    (property "Footprint" "kbd:D3_SMD" (id 2) (at 191.77 115.57 90)
+      (effects (font (size 1.27 1.27)) hide)
+    )
