File: ma8ic_split/ma8ic_split_69_left/ma8ic_split_69_left.kicad_pcb (KiCad board)
At the start: 2 copper layers, 166.3 x 125.7 mm, 133 parts, among them J1 USB_C_Receptacle, J2 MJ-4PP-9, J3 I2C, J4 SPI, SW1 SW_PUSH, SW10 SW_PUSH-kbd, SW11 SW_PUSH-kbd, SW12 SW_PUSH-kbd, SW13 SW_PUSH-kbd, SW14 SW_PUSH-kbd, SW15 SW_PUSH-kbd, SW16 SW_PUSH-kbd, SW17 SW_PUSH-kbd, SW18 SW_PUSH-kbd, SW19 SW_PUSH-kbd, SW2 SW_PUSH-kbd, SW20 SW_PUSH-kbd, SW21 SW_PUSH-kbd, SW22 SW_PUSH-kbd, SW23 SW_PUSH-kbd, SW24 SW_PUSH-kbd, SW25 SW_PUSH-kbd, SW26 SW_PUSH-kbd, SW27 SW_PUSH-kbd, SW28 SW_PUSH-kbd, SW29 SW_PUSH-kbd, SW3 SW_PUSH-kbd, SW30 SW_PUSH-kbd, SW31 SW_PUSH-kbd, SW32 SW_PUSH-kbd, SW33 SW_PUSH-kbd, SW4 SW_PUSH-kbd, SW5 SW_PUSH-kbd, SW6 SW_PUSH-kbd, SW7 SW_PUSH-kbd, SW8 SW_PUSH-kbd, SW9 SW_PUSH-kbd, U1 ATMEGA32U4, X1 CSTNE16M0V530000R0

Commit message: update
Parts:
- D1, D2, D3: footprint LED_SMD:LED_0603_1608Metric -> ma8ic_split_69:LED_0603_1608Metric
Changed lines of the file:
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@@
     )
   )
-  (footprint "LED_SMD:LED_0603_1608Metric" (layer "B.Cu")
+  (footprint "ma8ic_split_69:LED_0603_1608Metric" (layer "B.Cu")
     (at 207.406875 98.345625 10)
     (descr "LED SMD 0603 (1608 Metric), square (rectangular) end terminal, IPC_7351 nominal, (Body size source: http://www.tortai-tech.com/upload/download/2011102023233369053.pdf), generated with kicad-footprint-generator")
@@
     (property "Sheetname" "MCU")
     (attr smd)
-    (fp_text reference "D3" (at 0 1.43 10) (layer "B.Fab")
+    (fp_text reference "D3" (at 0 1.43 190) (layer "B.SilkS") hide
       (effects (font (size 1 1) (thickness 0.15)) (justify mirror))
     )
-    (fp_text value "BLUE" (at -3.66999 -5.241289 10) (layer "B.SilkS")
-      (effects (font (size 1 1) (thickness 0.15)) (justify right mirror))
+    (fp_text value "BLUE" (at 0 -1.43 190) (layer "B.Fab")
+      (effects (font (size 1 1) (thickness 0.15)) (justify mirror))
     )
-    (fp_text user "${REFERENCE}" (at 0 0 10) (layer "B.Fab")
+    (fp_text user "${REFERENCE}" (at -2.6 -0.1 190) (layer "B.Fab")
       (effects (font (size 0.4 0.4) (thickness 0.06)) (justify mirror))
     )
+    (fp_line (start -0.2 0.3) (end -0.2 -0.3) (layer "B.SilkS") (width 0.12))
     (fp_line (start 0.8 0.735) (end -1.485 0.735) (layer "B.SilkS") (width 0.12))
-    (fp_line (start -1.485 0.735) (end -1.485 -0.735) (layer "B.SilkS") (width 0.12))
+    (fp_line (start 0.2 0.3) (end 0.2 -0.3) (layer "B.SilkS") (width 0.12))
+    (fp_line (start -0.2 0) (end 0.2 0.3) (layer "B.SilkS") (width 0.12))
+    (fp_line (start 0.2 -0.3) (end -0.2 0) (layer "B.SilkS") (width 0.12))
     (fp_line (start -1.485 -0.735) (end 0.8 -0.735) (layer "B.SilkS") (width 0.12))
-    (fp_line (start -1.48 0.73) (end 1.48 0.73) (layer "B.CrtYd") (width 0.05))
-    (fp_line (start 1.48 0.73) (end 1.48 -0.73) (layer "B.CrtYd") (width 0.05))
+    (fp_line (start -1.485 0.735) (end -1.485 -0.735) (layer "B.SilkS") (width 0.12))
     (fp_line (start -1.48 -0.73) (end -1.48 0.73) (layer "B.CrtYd") (width 0.05))
+    (fp_line (start -1.48 0.73) (end 1.48 0.73) (layer "B.CrtYd") (width 0.05))
     (fp_line (start 1.48 -0.73) (end -1.48 -0.73) (layer "B.CrtYd") (width 0.05))
-    (fp_line (start -0.8 -0.4) (end 0.8 -0.4) (layer "B.Fab") (width 0.1))
-    (fp_line (start -0.8 0.1) (end -0.8 -0.4) (layer "B.Fab") (width 0.1))
-    (fp_line (start 0.8 0.4) (end -0.5 0.4) (layer "B.Fab") (width 0.1))
-    (fp_line (start -0.5 0.4) (end -0.8 0.1) (layer "B.Fab") (width 0.1))
+    (fp_line (start 1.48 0.73) (end 1.48 -0.73) (layer "B.CrtYd") (width 0.05))
     (fp_line (start 0.8 -0.4) (end 0.8 0.4) (layer "B.Fab") (width 0.1))
+    (fp_line (start -0.5 0.4) (end -0.8 0.1) (layer "B.Fab") (width 0.1))
+    (fp_line (start -0.8 0.1) (end -0.8 -0.4) (layer "B.Fab") (width 0.1))
     (pad "1" smd roundrect (at -0.7875 0 10) (size 0.875 0.95) (layers "B.Cu" "B.Paste" "B.Mask") (roundrect_rratio 0.25)
       (net 2 "GND") (pinfunction "K") (pintype "passive"))
@@
     )
   )
-  (footprint "LED_SMD:LED_0603_1608Metric" (layer "B.Cu")
+  (footprint "ma8ic_split_69:LED_0603_1608Metric" (layer "B.Cu")
     (at 206.454375 95.011875 10)
     (descr "LED SMD 0603 (1608 Metric), square (rectangular) end terminal, IPC_7351 nominal, (Body size source: http://www.tortai-tech.com/upload/download/2011102023233369053.pdf), generated with kicad-footprint-generator")
@@
     (property "Sheetname" "MCU")
     (attr smd)
-    (fp_text reference "D1" (at 0 1.43 10) (layer "B.Fab")
+    (fp_text reference "D1" (at 0 1.43 190) (layer "B.SilkS") hide
       (effects (font (size 1 1) (thickness 0.15)) (justify mirror))
     )
-    (fp_text value "RED" (at -2.897361 -4.13786 10) (layer "B.SilkS")
-      (effects (font (size 1 1) (thickness 0.15)) (justify right mirror))
+    (fp_text value "RED" (at 0 -1.43 190) (layer "B.Fab")
+      (effects (font (size 1 1) (thickness 0.15)) (justify mirror))
     )
-    (fp_text user "${REFERENCE}" (at 0 0 10) (layer "B.Fab")
+    (fp_text user "${REFERENCE}" (at -2.6 -0.1 190) (layer "B.Fab") hide
       (effects (font (size 0.4 0.4) (thickness 0.06)) (justify mirror))
     )
+    (fp_line (start -0.2 0.3) (end -0.2 -0.3) (layer "B.SilkS") (width 0.12))
+    (fp_line (start 0.2 0.3) (end 0.2 -0.3) (layer "B.SilkS") (width 0.12))
+    (fp_line (start -1.485 -0.735) (end 0.8 -0.735) (layer "B.SilkS") (width 0.12))
+    (fp_line (start -0.2 0) (end 0.2 0.3) (layer "B.SilkS") (width 0.12))
+    (fp_line (start 0.2 -0.3) (end -0.2 0) (layer "B.SilkS") (width 0.12))
     (fp_line (start -1.485 0.735) (end -1.485 -0.735) (layer "B.SilkS") (width 0.12))
     (fp_line (start 0.8 0.735) (end -1.485 0.735) (layer "B.SilkS") (width 0.12))
-    (fp_line (start -1.485 -0.735) (end 0.8 -0.735) (layer "B.SilkS") (width 0.12))
-    (fp_line (start 1.48 -0.73) (end -1.48 -0.73) (layer "B.CrtYd") (width 0.05))
     (fp_line (start 1.48 0.73) (end 1.48 -0.73) (layer "B.CrtYd") (width 0.05))
+    (fp_line (start 1.48 -0.73) (end -1.48 -0.73) (layer "B.CrtYd") (width 0.05))
     (fp_line (start -1.48 -0.73) (end -1.48 0.73) (layer "B.CrtYd") (width 0.05))
     (fp_line (start -1.48 0.73) (end 1.48 0.73) (layer "B.CrtYd") (width 0.05))
     (fp_line (start -0.8 0.1) (end -0.8 -0.4) (layer "B.Fab") (width 0.1))
-    (fp_line (start -0.5 0.4) (end -0.8 0.1) (layer "B.Fab") (width 0.1))
-    (fp_line (start -0.8 -0.4) (end 0.8 -0.4) (layer "B.Fab") (width 0.1))
     (fp_line (start 0.8 -0.4) (end 0.8 0.4) (layer "B.Fab") (width 0.1))
-    (fp_line (start 0.8 0.4) (end -0.5 0.4) (layer "B.Fab") (width 0.1))
+    (fp_line (start -0.5 0.4) (end -0.8 0.1) (layer "B.Fab") (width 0.1))
     (pad "1" smd roundrect (at -0.7875 0 10) (size 0.875 0.95) (layers "B.Cu" "B.Paste" "B.Mask") (roundrect_rratio 0.25)
       (net 5 "Net-(D1-Pad1)") (pinfunction "K") (pintype "passive"))
@@
     )
   )
-  (footprint "LED_SMD:LED_0603_1608Metric" (layer "B.Cu")
+  (footprint "ma8ic_split_69:LED_0603_1608Metric" (layer "B.Cu")
     (at 206.930625 96.67875 10)
     (descr "LED SMD 0603 (1608 Metric), square (rectangular) end terminal, IPC_7351 nominal, (Body size source: http://www.tortai-tech.com/upload/download/2011102023233369053.pdf), generated with kicad-footprint-generator")
@@
     (property "Sheetname" "MCU")
     (attr smd)
-    (fp_text reference "D2" (at 0 1.43 10) (layer "B.Fab")
+    (fp_text reference "D2" (at 0 1.43 190) (layer "B.SilkS") hide
       (effects (font (size 1 1) (thickness 0.15)) (justify mirror))
     )
-    (fp_text value "GREEN" (at -3.283675 -4.689574 10) (layer "B.SilkS")
-      (effects (font (size 1 1) (thickness 0.15)) (justify right mirror))
+    (fp_text value "GREEN" (at 0 -1.43 190) (layer "B.Fab")
+      (effects (font (size 1 1) (thickness 0.15)) (justify mirror))
     )
-    (fp_text user "${REFERENCE}" (at 0 0 10) (layer "B.Fab")
+    (fp_text user "${REFERENCE}" (at -2.6 -0.1 190) (layer "B.Fab") hide
       (effects (font (size 0.4 0.4) (thickness 0.06)) (justify mirror))
     )
-    (fp_line (start -1.485 -0.735) (end 0.8 -0.735) (layer "B.SilkS") (width 0.12))
     (fp_line (start -1.485 0.735) (end -1.485 -0.735) (layer "B.SilkS") (width 0.12))
+    (fp_line (start -1.485 -0.735) (end 0.8 -0.735) (layer "B.SilkS") (width 0.12))
     (fp_line (start 0.8 0.735) (end -1.485 0.735) (layer "B.SilkS") (width 0.12))
-    (fp_line (start 1.48 -0.73) (end -1.48 -0.73) (layer "B.CrtYd") (width 0.05))
+    (fp_line (start 0.2 0.3) (end 0.2 -0.3) (layer "B.SilkS") (width 0.12))
+    (fp_line (start 0.2 -0.3) (end -0.2 0) (layer "B.SilkS") (width 0.12))
+    (fp_line (start -0.2 0) (end 0.2 0.3) (layer "B.SilkS") (width 0.12))
+    (fp_line (start -0.2 0.3) (end -0.2 -0.3) (layer "B.SilkS") (width 0.12))
     (fp_line (start -1.48 0.73) (end 1.48 0.73) (layer "B.CrtYd") (width 0.05))
-    (fp_line (start 1.48 0.73) (end 1.48 -0.73) (layer "B.CrtYd") (width 0.05))
     (fp_line (start -1.48 -0.73) (end -1.48 0.73) (layer "B.CrtYd") (width 0.05))
-    (fp_line (start 0.8 0.4) (end -0.5 0.4) (layer "B.Fab") (width 0.1))
-    (fp_line (start -0.8 0.1) (end -0.8 -0.4) (layer "B.Fab") (width 0.1))
+    (fp_line (start 1.48 -0.73) (end -1.48 -0.73) (layer "B.CrtYd") (width 0.05))
+    (fp_line (start 1.48 0.73) (end 1.48 -0.73) (layer "B.CrtYd") (width 0.05))
     (fp_line (start 0.8 -0.4) (end 0.8 0.4) (layer "B.Fab") (width 0.1))
     (fp_line (start -0.5 0.4) (end -0.8 0.1) (layer "B.Fab") (width 0.1))
-    (fp_line (start -0.8 -0.4) (end 0.8 -0.4) (layer "B.Fab") (width 0.1))
+    (fp_line (start -0.8 0.1) (end -0.8 -0.4) (layer "B.Fab") (width 0.1))
     (pad "1" smd roundrect (at -0.7875 0 10) (size 0.875 0.95) (layers "B.Cu" "B.Paste" "B.Mask") (roundrect_rratio 0.25)
       (net 6 "Net-(D2-Pad1)") (pinfunction "K") (pintype "passive"))
