File: ma8ic_split/ma8ic_split_69_left/ma8ic_split_69_left.kicad_pcb (KiCad board)
At the start: 2 copper layers, 166.3 x 125.7 mm, 133 parts, among them J1 USB_C_Receptacle, J2 MJ-4PP-9, J3 OLED, J4 SPI, SW1 SW_PUSH, SW10 SW_PUSH-kbd, SW11 SW_PUSH-kbd, SW12 SW_PUSH-kbd, SW13 SW_PUSH-kbd, SW14 SW_PUSH-kbd, SW15 SW_PUSH-kbd, SW16 SW_PUSH-kbd, SW17 SW_PUSH-kbd, SW18 SW_PUSH-kbd, SW19 SW_PUSH-kbd, SW2 SW_PUSH-kbd, SW20 SW_PUSH-kbd, SW21 SW_PUSH-kbd, SW22 SW_PUSH-kbd, SW23 SW_PUSH-kbd, SW24 SW_PUSH-kbd, SW25 SW_PUSH-kbd, SW26 SW_PUSH-kbd, SW27 SW_PUSH-kbd, SW28 SW_PUSH-kbd, SW29 SW_PUSH-kbd, SW3 SW_PUSH-kbd, SW30 SW_PUSH-kbd, SW31 SW_PUSH-kbd, SW32 SW_PUSH-kbd, SW33 SW_PUSH-kbd, SW4 SW_PUSH-kbd, SW5 SW_PUSH-kbd, SW6 SW_PUSH-kbd, SW7 SW_PUSH-kbd, SW8 SW_PUSH-kbd, SW9 SW_PUSH-kbd, U1 ATMEGA32U4, X1 CSTNE16M0V530000R0

Commit message: update
Other:
- board text added: "ma8ic split rev0.2"
- board text removed: "ma8ic split rev0.1"
Changed lines of the file:
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@@
   (title_block
     (title "HatsuLight69")
-    (date "2023-01-02")
-    (rev "0.1")
+    (date "2023-03-09")
+    (rev "0.2")
     (company "kazmeegawa")
   )
@@
     (property "Sheetname" "MCU")
     (attr through_hole)
-    (fp_text reference "J1" (at -4.472573 -7.332416 180) (layer "F.SilkS")
+    (fp_text reference "J1" (at -4.472573 -7.332416 180) (layer "F.Fab")
       (effects (font (size 0.640654 0.640654) (thickness 0.15)))
     )
@@
     (effects (font (size 1 1) (thickness 0.15)) (justify left))
   )
-  (gr_text "ma8ic split rev0.1" (at 230.385845 100.012638 -270) (layer "F.SilkS")
+  (gr_text "ma8ic split rev0.2" (at 230.385845 100.012638 -270) (layer "F.SilkS")
     (effects (font (size 1 1) (thickness 0.15)))
   )
