File: ma8ic_split/ma8ic_split_69_left_bottom_plate/ma8ic_split_69_left_bottom_plate.kicad_pcb (KiCad board)
At the start: 2 copper layers, 166.3 x 125.7 mm, 133 parts, among them J1 USB_C_Receptacle, J2 MJ-4PP-9, J3 I2C, J4 SPI, SW1 SW_PUSH, SW10 SW_PUSH-kbd, SW11 SW_PUSH-kbd, SW12 SW_PUSH-kbd, SW13 SW_PUSH-kbd, SW14 SW_PUSH-kbd, SW15 SW_PUSH-kbd, SW16 SW_PUSH-kbd, SW17 SW_PUSH-kbd, SW18 SW_PUSH-kbd, SW19 SW_PUSH-kbd, SW2 SW_PUSH-kbd, SW20 SW_PUSH-kbd, SW21 SW_PUSH-kbd, SW22 SW_PUSH-kbd, SW23 SW_PUSH-kbd, SW24 SW_PUSH-kbd, SW25 SW_PUSH-kbd, SW26 SW_PUSH-kbd, SW27 SW_PUSH-kbd, SW28 SW_PUSH-kbd, SW29 SW_PUSH-kbd, SW3 SW_PUSH-kbd, SW30 SW_PUSH-kbd, SW31 SW_PUSH-kbd, SW32 SW_PUSH-kbd, SW33 SW_PUSH-kbd, SW4 SW_PUSH-kbd, SW5 SW_PUSH-kbd, SW6 SW_PUSH-kbd, SW7 SW_PUSH-kbd, SW8 SW_PUSH-kbd, SW9 SW_PUSH-kbd, U1 ATMEGA32U4, X1 CSTNE16M0V530000R0

Commit message: update
Routing:
- net Net-(D53-Pad2): track 35.1 -> 29.0 mm
- net GND: track 29.2 -> 29.6 mm, vias 140 -> 139
Changed lines of the file:
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@@
   (via (at 195.2625 38.1) (size 0.4) (drill 0.2) (layers "F.Cu" "B.Cu") (free) (net 2))
   (via (at 140.49375 116.68125) (size 0.4) (drill 0.2) (layers "F.Cu" "B.Cu") (free) (net 2))
-  (via (at 71.12 66.04) (size 0.605) (drill 0.3) (layers "F.Cu" "B.Cu") (free) (net 2))
   (via (at 59.53125 31.90875) (size 0.4) (drill 0.2) (layers "F.Cu" "B.Cu") (free) (net 2))
   (via (at 130.96875 126.20625) (size 0.4) (drill 0.2) (layers "F.Cu" "B.Cu") (free) (net 2))
@@
   (segment (start 186.588262 78.003262) (end 185.975625 77.390625) (width 0.1524) (layer "B.Cu") (net 2))
   (segment (start 185.2514 38.544332) (end 185.2514 38.5861) (width 0.1524) (layer "B.Cu") (net 2))
+  (segment (start 67.043904 67.220496) (end 67.043904 66.779823) (width 0.1524) (layer "B.Cu") (net 2))
   (segment (start 191.92875 38.57625) (end 192.643125 39.290625) (width 0.1524) (layer "B.Cu") (net 2))
   (segment (start 167.056488 105.282312) (end 167.056488 104.879855) (width 0.1524) (layer "B.Cu") (net 2))
@@
   (segment (start 146.959384 110.736266) (end 149.98845 107.7072) (width 0.1524) (layer "F.Cu") (net 4))
   (segment (start 146.959384 120.377145) (end 146.959384 110.736266) (width 0.1524) (layer "F.Cu") (net 4))
+  (segment (start 66.75 106.96875) (end 66.77355 106.9452) (width 0.1524) (layer "F.Cu") (net 4))
   (segment (start 150 107.69565) (end 149.98845 107.7072) (width 0.1524) (layer "F.Cu") (net 4))
   (segment (start 178.704401 103.632) (end 178.704401 106.6514) (width 0.1524) (layer "F.Cu") (net 4))
@@
   (segment (start 94.881432 85.829839) (end 84.305839 85.829839) (width 0.1524) (layer "B.Cu") (net 62))
   (segment (start 61.976 85.852) (end 61.976 73.914) (width 0.1524) (layer "F.Cu") (net 63))
-  (segment (start 59.944 67.818) (end 59.944 64.262) (width 0.1524) (layer "F.Cu") (net 63))
-  (segment (start 61.976 69.85) (end 59.944 67.818) (width 0.1524) (layer "F.Cu") (net 63))
-  (segment (start 61.976 73.914) (end 61.976 69.85) (width 0.1524) (layer "F.Cu") (net 63))
+  (segment (start 61.976 73.914) (end 68.58 67.31) (width 0.1524) (layer "F.Cu") (net 63))
   (via (at 61.976 85.852) (size 0.4) (drill 0.2) (layers "F.Cu" "B.Cu") (net 63))
-  (via (at 59.944 64.262) (size 0.605) (drill 0.3) (layers "F.Cu" "B.Cu") (net 63))
-  (segment (start 60.198 64.008) (end 66.548 64.008) (width 0.1524) (layer "B.Cu") (net 63))
-  (segment (start 66.548 64.008) (end 67.043904 64.503904) (width 0.1524) (layer "B.Cu") (net 63))
-  (segment (start 67.043904 64.503904) (end 67.043904 65.379823) (width 0.1524) (layer "B.Cu") (net 63))
+  (via (at 68.58 67.31) (size 0.4) (drill 0.2) (layers "F.Cu" "B.Cu") (net 63))
+  (segment (start 68.427823 65.379823) (end 67.043904 65.379823) (width 0.1524) (layer "B.Cu") (net 63))
   (segment (start 66.306408 85.829839) (end 61.998161 85.829839) (width 0.1524) (layer "B.Cu") (net 63))
   (segment (start 61.998161 85.829839) (end 61.976 85.852) (width 0.1524) (layer "B.Cu") (net 63))
-  (segment (start 59.944 64.262) (end 60.198 64.008) (width 0.1524) (layer "B.Cu") (net 63))
+  (segment (start 68.58 67.31) (end 68.58 65.532) (width 0.1524) (layer "B.Cu") (net 63))
+  (segment (start 68.58 65.532) (end 68.427823 65.379823) (width 0.1524) (layer "B.Cu") (net 63))
   (segment (start 61.543904 66.779823) (end 61.543904 67.690704) (width 0.1524) (layer "B.Cu") (net 64))
   (segment (start 82.296 64.008) (end 90.17 64.008) (width 0.1524) (layer "B.Cu") (net 64))
