File: ma8ic_split/ma8ic_split_69_left_bottom_plate/ma8ic_split_69_left_bottom_plate.kicad_sch (KiCad schematic)
At the start: 0 parts

Commit message: update
Other:
- removed sheet MCU
- removed sheet items
- removed sheet key_switch
