File: ma8ic_split/ma8ic_split_69_right/ma8ic_split_69_right.kicad_pcb (KiCad board)
At the start: 2 copper layers, 175.8 x 125.7 mm, 148 parts, among them J1 USB_C_Receptacle, J2 MJ-4PP-9, J3 I2C, J4 SPI, SW1 SW_PUSH, SW10 SW_PUSH-kbd, SW11 SW_PUSH-kbd, SW12 SW_PUSH-kbd, SW13 SW_PUSH-kbd, SW14 SW_PUSH-kbd, SW15 SW_PUSH-kbd, SW16 SW_PUSH-kbd, SW17 SW_PUSH-kbd, SW18 SW_PUSH-kbd, SW19 SW_PUSH-kbd, SW2 SW_PUSH-kbd, SW20 SW_PUSH-kbd, SW21 SW_PUSH-kbd, SW22 SW_PUSH-kbd, SW23 SW_PUSH-kbd, SW24 SW_PUSH-kbd, SW25 SW_PUSH-kbd, SW26 SW_PUSH-kbd, SW27 SW_PUSH-kbd, SW28 SW_PUSH-kbd, SW29 SW_PUSH-kbd, SW3 SW_PUSH-kbd, SW30 SW_PUSH-kbd, SW31 SW_PUSH-kbd, SW32 SW_PUSH-kbd, SW33 SW_PUSH-kbd, SW34 SW_PUSH-kbd, SW35 SW_PUSH-kbd, SW36 SW_PUSH-kbd, SW37 SW_PUSH-kbd, SW38 SW_PUSH-kbd, SW4 SW_PUSH-kbd, SW5 SW_PUSH-kbd, SW6 SW_PUSH-kbd, SW7 SW_PUSH-kbd, SW8 SW_PUSH-kbd, SW9 SW_PUSH-kbd, U1 ATMEGA32U4, X1 CSTNE16M0V530000R0

Commit message: update
Parts:
- D10, D11, D12, D13, D14, D15, D16, D17, D19, D20, D21, D22, D23, D24, D26, D27, D28, D29, D30, D31, D34, D35, D36, D37, D38, D39, D4, D5, D6, D7, D8, D9: footprint kbd:D3_SMD_v2 -> ma8ic_split_69:D3_SMD_v2
- D41, D42, D43, D44, D45, D46, D47, D48, D49, D50, D51, D52, D53, D54, D56, D57, D58, D59, D60, D61, D63, D64, D65, D66, D67, D68, D71, D72, D73, D74, D75, D76: footprint kbd:YS-SK6812MINI-E -> ma8ic_split_69:YS-SK6812MINI-E
- J1: footprint HatsuLight69:HRS_CX70M-24P1 -> ma8ic_split_69:HRS_CX70M-24P1
- J4: footprint Connector_PinHeader_2.54mm:PinHeader_1x07_P2.54mm_Vertical -> ma8ic_split_69:PinSocket_1x07_P2.54mm_Vertical
- SW1: footprint kbd:ResetSW_1side -> ma8ic_split_69:ResetSW_1side
- SW17, SW2, SW36: footprint ma8ic_split_69:ChocV1_V2_Hotswap_1.5u -> ma8ic_split_69:ChocV1_V2_Hotswap
- SW38: footprint ma8ic_split_69:ChocV1_V2_Hotswap_2u -> ma8ic_split_69:ChocV1_V2_Hotswap
- U1: footprint ma8ic_split_69:TQFP-44_10x10mm_P0.8mm -> ma8ic_split_69:QFN-44-1EP_7x7mm_P0.5mm_EP5.2x5.2mm
Routing:
- net /MCU/D+: track 50.3 -> 58.2 mm
- net VCC: track 1137.6 -> 1145.3 mm, vias 76 -> 81
- net /MCU/D-: track 50.0 -> 55.9 mm
- net Net-(R7-Pad1): track 2.42 -> 6.70 mm
- net Net-(R8-Pad2): track 30.9 -> 35.0 mm
- net DATA: track 33.2 -> 37.0 mm
- net GND: track 29.6 -> 32.9 mm, vias 263 -> 269
- net COL1: track 197.9 -> 200.7 mm
- net COL0: track 209.8 -> 212.5 mm
- net COL2: track 179.4 -> 182.1 mm
- net NCS: track 84.5 -> 87.2 mm
- net ROW4: track 220.4 -> 223.0 mm
- net /MCU/XTAL1: track 3.36 -> 5.85 mm
- net ROW3: track 164.3 -> 166.8 mm
- net COL3: track 153.6 -> 156.1 mm
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Other:
- board text added: "ma8ic split rev0.2"
- board text removed: "ma8ic split rev0.1"
