File: ma8ic_split/ma8ic_split_69_right/items.kicad_sch (KiCad schematic)
At the start: 34 parts, among them J3 OLED, J4 SPI

Commit message: update
Parts:
- added D55, D62, D69, D70, D77: SK6812MINI, ma8ic_split_69:YS-SK6812MINI-E, symbol ma8ic_split_69:YS-SK6812MINI-E
- renumbered D36 to D41, D37 to D42, D38 to D43, D39 to D44, D40 to D45, D41 to D46, D42 to D47, D43 to D48, D44 to D49, D45 to D50, D46 to D51, D47 to D52, D48 to D53, D49 to D54, D50 to D56, D51 to D57, D52 to D58, D53 to D59, D54 to D60, D55 to D61, D56 to D63, D57 to D64, D58 to D65, D59 to D66, D60 to D67, D61 to D68, D62 to D71, D63 to D72, D64 to D73, D65 to D74, D66 to D75, D67 to D76
Connections:
- net GND: now also D55.3 (VSS), D62.3 (VSS), D69.3 (VSS), D70.3 (VSS), D77.3 (VSS)
- net VCC: now also D55.1 (VDD), D62.1 (VDD), D69.1 (VDD), D70.1 (VDD), D77.1 (VDD)
- net at D61.2 (DOUT): now also D62.4 (DIN); no longer D63.4 (DIN)
- net at D56.4 (DIN): now also D55.2 (DOUT); no longer D54.2 (DOUT)
- net at D68.2 (DOUT): now also D69.4 (DIN); no longer D71.4 (DIN)
- net at D76.2 (DOUT): now also D77.4 (DIN)
- new net: D54.2 (DOUT), D55.4 (DIN)
- new net: D70.2 (DOUT), D71.4 (DIN)
- new net: D69.2 (DOUT), D70.4 (DIN)
- new net: D62.2 (DOUT), D63.4 (DIN)

Commit message: update
Parts:
- D41, D42, D43, D44, D45, D46, D47, D48, D49, D50, D51, D52, D53, D54, D55, D56, D57, D58, D59, D60, D61, D62, D63, D64, D65, D66, D67, D68, D69, D70, D71, D72, D73, D74, D75, D76, D77: LCSC (none) -> C5149201
