File: ma8ic_split/ma8ic_split_69_pcbs/key_switch_left.kicad_sch (KiCad schematic)
At the start: 64 parts, among them SW10 SW_PUSH-kbd, SW11 SW_PUSH-kbd, SW12 SW_PUSH-kbd, SW13 SW_PUSH-kbd, SW14 SW_PUSH-kbd, SW15 SW_PUSH-kbd, SW16 SW_PUSH-kbd, SW17 SW_PUSH-kbd, SW18 SW_PUSH-kbd, SW19 SW_PUSH-kbd, SW2 SW_PUSH-kbd, SW20 SW_PUSH-kbd, SW21 SW_PUSH-kbd, SW22 SW_PUSH-kbd, SW23 SW_PUSH-kbd, SW24 SW_PUSH-kbd, SW25 SW_PUSH-kbd, SW26 SW_PUSH-kbd, SW27 SW_PUSH-kbd, SW28 SW_PUSH-kbd, SW29 SW_PUSH-kbd, SW3 SW_PUSH-kbd, SW30 SW_PUSH-kbd, SW31 SW_PUSH-kbd, SW32 SW_PUSH-kbd, SW33 SW_PUSH-kbd, SW4 SW_PUSH-kbd, SW5 SW_PUSH-kbd, SW6 SW_PUSH-kbd, SW7 SW_PUSH-kbd, SW8 SW_PUSH-kbd, SW9 SW_PUSH-kbd

Commit message: update
Connections:
- net COL0: now also SW16.2, SW2.2, SW22.2, SW28.2, SW9.2; no longer SW16.1, SW2.1, SW22.1, SW28.1, SW9.1
- net COL1: now also SW10.2, SW17.2, SW23.2, SW29.2, SW3.2; no longer SW10.1, SW17.1, SW23.1, SW29.1, SW3.1
- net COL2: now also SW11.2, SW18.2, SW24.2, SW30.2, SW4.2; no longer SW11.1, SW18.1, SW24.1, SW30.1, SW4.1
- net COL3: now also SW12.2, SW19.2, SW25.2, SW31.2, SW5.2; no longer SW12.1, SW19.1, SW25.1, SW31.1, SW5.1
- net COL4: now also SW13.2, SW20.2, SW26.2, SW32.2, SW6.2; no longer SW13.1, SW20.1, SW26.1, SW32.1, SW6.1
- net COL5: now also SW14.2, SW21.2, SW27.2, SW33.2, SW7.2; no longer SW14.1, SW21.1, SW27.1, SW33.1, SW7.1
- net COL6: now also SW15.2, SW8.2; no longer SW15.1, SW8.1
- net at D21.2 (A): now also SW19.1; no longer SW19.2
- net at D24.2 (A): now also SW22.1; no longer SW22.2
- net at D19.2 (A): now also SW17.1; no longer SW17.2
- net at D27.2 (A): now also SW25.1; no longer SW25.2
- net at D28.2 (A): now also SW26.1; no longer SW26.2
- net at D32.2 (A): now also SW30.1; no longer SW30.2
- net at D10.2 (A): now also SW8.1; no longer SW8.2
- net at D33.2 (A): now also SW31.1; no longer SW31.2
- net at D26.2 (A): now also SW24.1; no longer SW24.2
- net at D17.2 (A): now also SW15.1; no longer SW15.2
- net at D34.2 (A): now also SW32.1; no longer SW32.2
- net at D30.2 (A): now also SW28.1; no longer SW28.2
- net at D35.2 (A): now also SW33.1; no longer SW33.2
- net at D7.2 (A): now also SW5.1; no longer SW5.2
- net at D31.2 (A): now also SW29.1; no longer SW29.2
- net at D20.2 (A): now also SW18.1; no longer SW18.2
- net at D23.2 (A): now also SW21.1; no longer SW21.2
- net at D13.2 (A): now also SW11.1; no longer SW11.2
- net at D12.2 (A): now also SW10.1; no longer SW10.2
- net at D11.2 (A): now also SW9.1; no longer SW9.2
- net at D5.2 (A): now also SW3.1; no longer SW3.2
- net at D14.2 (A): now also SW12.1; no longer SW12.2
- net at D22.2 (A): now also SW20.1; no longer SW20.2
- net at D29.2 (A): now also SW27.1; no longer SW27.2
- net at D25.2 (A): now also SW23.1; no longer SW23.2
- net at D16.2 (A): now also SW14.1; no longer SW14.2
- net at D18.2 (A): now also SW16.1; no longer SW16.2
- net at D8.2 (A): now also SW6.1; no longer SW6.2
- net at D6.2 (A): now also SW4.1; no longer SW4.2
- net at D4.2 (A): now also SW2.1; no longer SW2.2
- net at D9.2 (A): now also SW7.1; no longer SW7.2
- net at D15.2 (A): now also SW13.1; no longer SW13.2
Other:
- moved on the sheet: SW10, SW11, SW12, SW13, SW14, SW15, SW16, SW17, SW18, SW19, SW2, SW20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
